File: PCB/shield/kicad/mailboxguard_shield.kicad_sch (KiCad schematic)
At the start: 9 parts, among them Q1 MMBT3904, SW1 BUZ_STOP

Commit message: Updating GERBER files for shield
Parts:
- R1: value 1K -> 470 - 1K
Changed lines of the file:
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@@
+		)
+	)
+	(text_box "Une valeur de 300R serait bien (5mA de consommation avec un courrant de 1.8 (mesuré pour diode verte) J'ai seulement 470R en 1206"
+		(exclude_from_sim no)
+		(at 127 109.22 0)
+		(size 21.59 17.78)
+		(stroke
+			(width 0)
+			(type default)
+		)
+		(fill
+			(type none)
+		)
+		(effects
+			(font
+				(size 1.27 1.27)
+			)
+			(justify left top)
 		)
 	)
@@
 			)
 		)
-		(property "Value" "1K"
+		(property "Value" "470 - 1K"
 			(at 121.92 114.2999 0)
 			(effects
