File: PCB/shield/kicad/mailboxguard_shield.kicad_pcb (KiCad board)
At the start: 2 copper layers, 28 x 53.5 mm, 9 parts, among them Q1 MMBT3904, SW1 BUZ_STOP

Commit message: Updating GERBER files for shield
Parts:
- R1: value 1K -> 470 - 1K
Changed lines of the file:
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@@
 		(pad_to_mask_clearance 0)
 		(allow_soldermask_bridges_in_footprints no)
+		(aux_axis_origin 69 82.5)
 		(grid_origin 69 82.5)
 		(pcbplotparams
@@
 			)
 		)
-		(property "Value" "1K"
+		(property "Value" "470 - 1K"
 			(at 0 1.82 90)
 			(layer "F.Fab")

Commit message: Updating SVG files for PCB
Other:
- board text added: "03/24"
- board text added: "MailboxguardShield"
Changed lines of the file:
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@@
 		(layer "Edge.Cuts")
+	)
+	(gr_text "MailboxguardShield"
+		(at 88.25 49.75 90)
+		(layer "B.SilkS")
+		(effects
+			(font
+				(size 2 2)
+				(thickness 0.4)
+				(bold yes)
+			)
+			(justify left bottom mirror)
+		)
+	)
+	(gr_text "03/24"
+		(at 91.25 60 90)
+		(layer "B.SilkS")
+		(effects
+			(font
+				(size 1 1)
+				(thickness 0.1)
+			)
+			(justify left bottom mirror)
+		)
 	)
 	(segment
